File: KiCad/V1/PWM_Generator.kicad_sch (KiCad schematic)
At the start: 0 parts

Commit message: kicad scematic
Parts:
- added C2: 20p, symbol Device:C
- added C3, C4, C5, C6, C7, C8: C, symbol Device:C
- added R2, R3: 250, symbol Device:R
- added R4, R5: 100, symbol Device:R
- added R6, R7: 0, symbol Device:R
- added RV1: R_Potentiometer, symbol Device:R_Potentiometer
- added RV2: 1k, symbol Device:R_Potentiometer
- added U3, U4: OPA2677IDDA, DDA8_3X2P49, symbol 2024-11-17_16-46-04:OPA2677IDDA
Connections:
- new net: R4.2, R5.1, U3.2 (INA-)
- new net: RV2.2, U4.3 (INA+)
- new net: R2.2, R3.2, U3.1 (OUTA)
- new net: R3.1, RV1.1, U3.3 (INA+)
- new net: C2.1, R2.1, U3.6 (INB-)
- new net: C2.2, RV1.2, U3.7 (OUTB), U4.2 (INA-)
- new net: R6.1, R7.2, U4.4 (VS-)
- new net +5V: C3.2, C4.2, C5.2, C6.2, C7.2, C8.2, R4.1, U3.8 (VS+), U4.7 (OUTB)
- new net -1V: R7.1
- new net GND: C3.1, C4.1, C5.1, C6.1, C7.1, C8.1, R5.2, R6.2, RV2.3, U3.4 (VS-), U3.5 (INB+), U3.EPAD, U4.8 (VS+)
- new net V_reff: RV2.1
