File: KiCad/V1/_autosave-V1.kicad_pcb (KiCad board)
At the start: 4 copper layers, 130.8 x 93.1 mm, 84 parts, among them Q1 Q_NMOS_GSD, Q2 Q_NMOS_GSD, U1 LMG1210RVRR, U2 OPA2677IDDA, U3 OPA2677IDDA, U4 OPA859QDSGRQ1, U5 OPA859QDSGRQ1, U6 OPA859QDSGRQ1

Commit message: V1 pcb almost done
Parts:
- moved RdtL1 0.45 mm to (118.0, 42.5)
- moved C3 0.34 mm to (120.7, 42.5)
- moved C14 0.20 mm to (139.0, 55.5)
- moved C7 0.08 mm to (150.1, 57.6)
Connections:
- Q1 pad 3: /VDD_PWM_Big -> /HS1
- Q1 pad 4: (no net) -> /VDD_PWM_Big
- Q1 pad 5: (no net) -> /HS1
- Q1 pad 6: (no net) -> /HS1
- Q2 pad 3: /HS1 -> GND
- Q2 pad 5: (no net) -> GND
- Q2 pad 6: (no net) -> GND
- VDD_PWM_BIG3 pad 1: /-I_OUT -> GND
Routing:
- net GND: track 19.2 -> 21.8 mm, vias 53 -> 69
- net Net-(U1-DHL): track 4.12 -> 5.11 mm
- net /VDD10: track 21.8 -> 21.1 mm
- net /EN1: track 44.0 -> 44.6 mm
