File: KiCad/V1/V1.kicad_sch (KiCad schematic)
At the start: 85 parts, among them Q1 Q_NMOS_GSD, Q2 Q_NMOS_GSD, T1 Transformer_1P_1S, U1 LMG1210RVRR, U2 OPA2677IDDA, U3 OPA2677IDDA, U4 OPA859QDSGRQ1, U5 OPA859QDSGRQ1, U6 OPA859QDSGRQ1

Commit message: V1 done
Parts:
- removed EN1: MountingHole_Pad, TestPoint:TestPoint_THTPad_D2.5mm_Drill1.2mm, symbol Mechanical:MountingHole_Pad
- T1: footprint (none) -> MyFootprints:MyTransformer
- renumbered EN1 to EN1_coax1, PWM_External to PWM_External1, Pre_FilterV_ref to Pre_FilterV_ref1, Pre_FilterV_duffsense to V_duffsense1
Connections:
- net -I_OUT is gone; now on net GND: VDD_PWM_BIG3.1
- net +I_OUT: now also C13.2, T1.1 (AA)
- net at R8.1, R_shutn1.2: now also T1.4 (SB); no longer T1.3 (SA)
- net at R8.8, R_shutn1.1: now also T1.3 (SA); no longer T1.4 (SB)
- net at L2.2: now also T1.2 (AB); no longer T1.1 (AA)
- removed net OUT: C13.2, T1.2 (AB)
Other:
- moved on the sheet: D1, D2, T1
Changed lines of the file:
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@@
 	(wire
 		(pts
-			(xy 320.04 175.26) (xy 320.04 179.07)
+			(xy 320.04 175.26) (xy 320.04 180.34)
 		)
 		(stroke
@@
 	(wire
 		(pts
-			(xy 298.45 39.37) (xy 304.8 39.37)
+			(xy 294.64 39.37) (xy 304.8 39.37)
 		)
 		(stroke
@@
 	(wire
 		(pts
+			(xy 320.04 172.72) (xy 320.04 175.26)
+		)
+		(stroke
+			(width 0)
+			(type default)
+		)
+	)
+	(wire
+		(pts
 			(xy 120.65 138.43) (xy 120.65 135.89)
 		)
@@
 	(wire
 		(pts
+			(xy 327.66 172.72) (xy 327.66 175.26)
+		)
+		(stroke
+			(width 0)
+			(type default)
+		)
+	)
+	(wire
+		(pts
 			(xy 168.91 74.93) (xy 179.07 74.93)
 		)
@@
 	(wire
 		(pts
-			(xy 327.66 175.26) (xy 327.66 179.07)
+			(xy 327.66 175.26) (xy 327.66 180.34)
 		)
 		(stroke
@@
 	)
 	(label "V_diffsense"
-		(at 298.45 39.37 0)
+		(at 294.64 39.37 0)
 		(fields_autoplaced yes)
 		(effects
@@
 		)
 	)
-	(label "OUT"
+	(label "+I_OUT"
 		(at 101.6 26.67 0)
 		(fields_autoplaced yes)
@@
 		(dnp no)
 		(fields_autoplaced yes)
-		(property "Reference" "EN1"
+		(property "Reference" "EN1_coax1"
 			(at 339.09 67.6031 0)
 			(effects
@@
 			(project "V1"
 				(path "/009e4554-048b-4d13-979d-7fdd312db04d"
-					(reference "EN1")
+					(reference "EN1_coax1")
 					(unit 1)
 				)
@@
 		(dnp no)
 		(fields_autoplaced yes)
-		(property "Reference" "PWM_External"
+		(property "Reference" "PWM_External1"
 			(at 337.82 35.8531 0)
 			(effects
@@
 			(project ""
 				(path "/009e4554-048b-4d13-979d-7fdd312db04d"
-					(reference "PWM_External")
+					(reference "PWM_External1")
 					(unit 1)
 				)
@@
 		(on_board yes)
 		(dnp no)
-		(property "Reference" "Pre_FilterV_duffsense"
+		(property "Reference" "V_duffsense1"
 			(at 312.166 40.894 0)
 			(effects
@@
 			(project "V1"
 				(path "/009e4554-048b-4d13-979d-7fdd312db04d"
-					(reference "Pre_FilterV_duffsense")
+					(reference "V_duffsense1")
 					(unit 1)
 				)
@@
 	)
 	(symbol
+		(lib_id "power:GND")
+		(at 389.89 55.88 270)
+		(unit 1)
+		(exclude_from_sim no)
+		(in_bom yes)
+		(on_board yes)
+		(dnp no)
+		(fields_autoplaced yes)
+		(property "Reference" "#PWR020"
+			(at 383.54 55.88 0)
+			(effects
+				(font
+					(size 1.27 1.27)
+				)
+				(hide yes)
+			)
+		)
+		(property "Value" "GND"
+			(at 386.08 55.8799 90)
+			(effects
+				(font
+					(size 1.27 1.27)
+				)
+				(justify right)
+			)
+		)
+		(property "Footprint" ""
+			(at 389.89 55.88 0)
+			(effects
+				(font
+					(size 1.27 1.27)
+				)
+				(hide yes)
+			)
+		)
+		(property "Datasheet" ""
+			(at 389.89 55.88 0)
+			(effects
+				(font
+					(size 1.27 1.27)
+				)
+				(hide yes)
+			)
+		)
+		(property "Description" "Power symbol creates a global label with name \"GND\" , ground"
+			(at 389.89 55.88 0)
+			(effects
+				(font
+					(size 1.27 1.27)
+				)
+				(hide yes)
+			)
+		)
+		(pin "1"
+		)
+		(instances
+			(project "V1"
+				(path "/009e4554-048b-4d13-979d-7fdd312db04d"
+					(reference "#PWR020")
+					(unit 1)
+				)
+			)
+		)
+	)
+	(symbol
 		(lib_id "Device:C")
 		(at 95.25 223.52 180)
@@
 		(lib_name "D_Schottky_2")
 		(lib_id "Device:D_Schottky")
-		(at 323.85 179.07 180)
+		(at 323.85 180.34 180)
 		(unit 1)
 		(exclude_from_sim no)
@@
 		(fields_autoplaced yes)
 		(property "Reference" "D2"
-			(at 324.1675 172.72 0)
+			(at 324.1675 173.99 0)
 			(effects
 				(font
@@
 		)
 		(property "Value" "D_Schottky"
-			(at 324.1675 175.26 0)
+			(at 324.1675 176.53 0)
 			(effects
 				(font
@@
 		)
 		(property "Footprint" "Package_TO_SOT_SMD:SOT-323_SC-70"
-			(at 323.596 182.372 0)
+			(at 323.596 183.642 0)
 			(effects
 				(font
@@
 		)
 		(property "Datasheet" "~"
-			(at 323.85 179.07 0)
+			(at 323.85 180.34 0)
 			(effects
 				(font
@@
 		)
 		(property "Description" "Schottky diode"
-			(at 323.85 181.102 0)
+			(at 323.85 182.372 0)
 			(effects
 				(font
@@
 		)
 		(property "Sim.Device" ""
-			(at 323.85 179.07 0)
+			(at 323.85 180.34 0)
 			(effects
 				(font
@@
 		)
 		(property "Sim.Pins" ""
-			(at 323.85 179.07 0)
+			(at 323.85 180.34 0)
 			(effects
 				(font
@@
 		)
 		(property "Sim.Type" ""
-			(at 323.85 179.07 0)
+			(at 323.85 180.34 0)
 			(effects
 				(font
@@
 	(symbol
 		(lib_id "Device:Transformer_1P_1S")
-		(at 67.31 60.96 90)
-		(mirror x)
+		(at 67.31 60.96 270)
 		(unit 1)
 		(exclude_from_sim no)
@@
 		(on_board yes)
 		(dnp no)
-		(fields_autoplaced yes)
 		(property "Reference" "T1"
-			(at 73.66 59.7026 90)
+			(at 60.96 59.7026 90)
 			(effects
 				(font
@@
 		)
 		(property "Value" "Transformer_1P_1S"
-			(at 73.66 62.2426 90)
+			(at 60.96 62.2426 90)
 			(effects
 				(font
@@
 			)
 		)
-		(property "Footprint" ""
+		(property "Footprint" "MyFootprints:MyTransformer"
 			(at 67.31 60.96 0)
 			(effects
@@
 		(lib_name "D_Schottky_1")
 		(lib_id "Device:D_Schottky")
-		(at 323.85 175.26 180)
+		(at 323.85 172.72 180)
 		(unit 1)
 		(exclude_from_sim no)
@@
 		(fields_autoplaced yes)
 		(property "Reference" "D1"
-			(at 324.1675 168.91 0)
+			(at 324.1675 166.37 0)
 			(effects
 				(font
@@
 		)
 		(property "Value" "D_Schottky"
-			(at 324.1675 171.45 0)
+			(at 324.1675 168.91 0)
 			(effects
 				(font
@@
 		)
 		(property "Footprint" "Package_TO_SOT_SMD:SOT-323_SC-70"
-			(at 323.596 178.562 0)
+			(at 323.596 176.022 0)
 			(effects
 				(font
@@
 		)
 		(property "Datasheet" "~"
-			(at 323.85 175.26 0)
+			(at 323.85 172.72 0)
 			(effects
 				(font
@@
 		)
 		(property "Description" "Schottky diode"
-			(at 323.85 177.292 0)
+			(at 323.85 174.752 0)
 			(effects
 				(font
@@
 		)
 		(property "Sim.Device" ""
-			(at 323.85 175.26 0)
+			(at 323.85 172.72 0)
 			(effects
 				(font
@@
 		)
 		(property "Sim.Pins" ""
-			(at 323.85 175.26 0)
+			(at 323.85 172.72 0)
 			(effects
 				(font
@@
 		)
 		(property "Sim.Type" ""
-			(at 323.85 175.26 0)
+			(at 323.85 172.72 0)
 			(effects
 				(font
@@
 	)
 	(symbol
-		(lib_id "Mechanical:MountingHole_Pad")
-		(at 229.87 219.71 180)
-		(unit 1)
-		(exclude_from_sim yes)
-		(in_bom no)
-		(on_board yes)
-		(dnp no)
-		(property "Reference" "EN1"
-			(at 232.41 219.7099 0)
-			(effects
-				(font
-					(size 1.27 1.27)
-				)
-				(justify right)
-			)
-		)
-		(property "Value" "MountingHole_Pad"
-			(at 232.41 222.2499 0)
-			(effects
-				(font
-					(size 1.27 1.27)
-				)
-				(justify right)
-			)
-		)
-		(property "Footprint" "TestPoint:TestPoint_THTPad_D2.5mm_Drill1.2mm"
-			(at 229.87 219.71 0)
-			(effects
-				(font
-					(size 1.27 1.27)
-				)
-				(hide yes)
-			)
-		)
-		(property "Datasheet" "~"
-			(at 229.87 219.71 0)
-			(effects
-				(font
-					(size 1.27 1.27)
-				)
-				(hide yes)
-			)
-		)
-		(property "Description" "Mounting Hole with connection"
-			(at 229.87 219.71 0)
-			(effects
-				(font
-					(size 1.27 1.27)
-				)
-				(hide yes)
-			)
-		)
-		(property "Sim.Device" ""
-			(at 229.87 219.71 0)
-			(effects
-				(font
-					(size 1.27 1.27)
-				)
-				(hide yes)
-			)
-		)
-		(property "Sim.Pins" ""
-			(at 229.87 219.71 0)
-			(effects
-				(font
-					(size 1.27 1.27)
-				)
-				(hide yes)
-			)
-		)
-		(property "Sim.Type" ""
-			(at 229.87 219.71 0)
-			(effects
-				(font
-					(size 1.27 1.27)
-				)
-				(hide yes)
-			)
-		)
-		(pin "1"
-		)
-		(instances
-			(project ""
-				(path "/009e4554-048b-4d13-979d-7fdd312db04d"
-					(reference "EN1")
-					(unit 1)
-				)
-			)
-			(project "MosTest"
-				(path "/e10a9314-4860-4bd8-b877-dab830b8ef59"
-					(reference "EN1")
-					(unit 1)
-				)
-			)
-		)
-	)
-	(symbol
 		(lib_id "Device:R")
 		(at 242.57 198.12 90)
@@
 		(on_board yes)
 		(dnp no)
-		(property "Reference" "Pre_FilterV_ref"
+		(property "Reference" "Pre_FilterV_ref1"
 			(at 307.34 15.494 0)
 			(effects
@@
 			(project "V1"
 				(path "/009e4554-048b-4d13-979d-7fdd312db04d"
-					(reference "Pre_FilterV_ref")
+					(reference "Pre_FilterV_ref1")
 					(unit 1)
 				)

Commit message: Fixed GanfetPad clerance
Parts:
- C17: footprint Capacitor_SMD:C_0402_1005Metric -> Capacitor_SMD:C_0805_2012Metric
Changed lines of the file:
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@@
 			)
 		)
-		(property "Footprint" "Capacitor_SMD:C_0402_1005Metric"
+		(property "Footprint" "Capacitor_SMD:C_0805_2012Metric"
 			(at 366.7252 180.34 0)
 			(effects
